Commit message: upd: gps fixed, 1d lidar added

File: ifo_description/materials/materials.xacro (robot description, xacro)
@@ -4,3 +4,6 @@
         <color rgba="1 1 1 1"/>
     </material>
+    <material name="red">
+        <color rgba="1 0 0 1"/>
+    </material>
 </robot>

File: ifo_description/urdf/ifo.xacro (robot description, xacro)
@@ -6,4 +6,5 @@
     <xacro:arg name="namespace" default=""/>
     <xacro:arg name="camera" default="true"/>
+    <xacro:arg name="lidar" default="true"/>
     <!-- Include base -->
     <xacro:include filename="$(find ifo_description)/urdf/ifo_base.xacro" />
@@ -16,3 +17,25 @@
         </xacro:realsense_d435i>
     </xacro:if>
+    <!-- Include 1D LIDAR at the bottom -->
+    <xacro:if value="$(arg lidar)">
+        <xacro:include filename="$(find ifo_description)/urdf/lidar.xacro" />
+        <xacro:lidar parent="base_link" name="$(arg namespace)/laser">
+            <origin xyz="0 0 0" rpy="0 0 0" />
+        </xacro:lidar>
+    </xacro:if>
+    <!-- <include>
+      <uri>model://fpv_cam</uri>
+      <pose>0 0 0 0 0 0</pose>
+    </include> -->
+    <!-- <joint name="fpv_cam_joint" type="fixed">
+      <child>fpv_cam::link</child>
+      <parent>iris::base_link</parent>
+      <axis>
+        <xyz>0 0 1</xyz>
+        <limit>
+          <upper>0</upper>
+          <lower>0</lower>
+        </limit>
+      </axis>
+    </joint> -->
 </robot>

File: ifo_description/urdf/ifo_base.xacro (robot description, xacro)
@@ -33,5 +33,5 @@
       </collision>
       <inertial>
-          <mass value="1.5"/>
+          <mass value="1.5" />
           <inertia
             ixx="0.029125" ixy="0.0" ixz="0.0"
@@ -68,7 +68,32 @@
       <visual>
         <geometry>
-          <cylinder length="0.01" radius="0.1"/>
-        </geometry>
-      </visual>
+            <cylinder length="0.01" radius="0.1"/>
+        </geometry>
+      </visual>
+      <inertial>
+        <mass value="0.005" />
+        <inertia
+          ixx="9.75e-07" ixy="0.0" ixz="0.0"
+          iyy="0.000273104" iyz="0.0"
+          izz="0.000274004"/>
+      </inertial>
+      <pose>0.13 -0.22 0.023 0 0 0</pose>
+      <collision name='rotor_0_collision'>
+        <pose>0 0 0 0 0 0</pose>
+        <geometry>
+          <cylinder>
+            <length>0.005</length>
+            <radius>0.128</radius>
+          </cylinder>
+        </geometry>
+        <surface>
+          <contact>
+            <ode/>
+          </contact>
+          <friction>
+            <ode/>
+          </friction>
+        </surface>
+      </collision>
     </link>
     <joint name="rotor_0_joint" type="revolute">
@@ -79,19 +104,192 @@
       <limit lower="-1e+16" upper="+1e+16" effort="0" velocity="0"/>
     </joint>
-    <gazebo>
-      <link name='rotor_0'>
-        <pose>0.13 -0.22 0.023 0 0 0</pose>
-        <inertial>
-          <mass>0.005</mass>
-          <inertia>
-            <ixx>9.75e-07</ixx>
-            <ixy>0</ixy>
-            <ixz>0</ixz>
-            <iyy>0.000273104</iyy>
-            <iyz>0</iyz>
-            <izz>0.000274004</izz>
-          </inertia>
-        </inertial>
-        <collision name='rotor_0_collision'>
+    <gazebo reference="rotor_0">
+      <gravity>1</gravity>
+      <visual name='rotor_0_visual'>
+          <pose>0 0 0 0 0 0</pose>
+          <geometry>
+              <mesh>
+                  <scale>1 1 1</scale>
+                  <uri>$(find ifo_description)/meshes/iris_prop_cw.dae</uri>
+              </mesh>
+          </geometry>
+          <material>
+              <script>
+                  <name>Gazebo/Blue</name>
+                  <uri>file://media/materials/scripts/gazebo.material</uri>
+              </script>
+          </material>
+      </visual>
+      <velocity_decay/>
+    </gazebo>
+	<gazebo reference="rotor_0_joint">
+		<dynamics>
+		    <spring_reference>0</spring_reference>
+		    <spring_stiffness>0</spring_stiffness>
+		</dynamics>
+		<use_parent_model_frame>1</use_parent_model_frame>
+	</gazebo>
+    <!-- ===================================================================== -->
+    <!--                               ROTOR 1                                 -->
+    <!-- ===================================================================== -->
+    <!-- For each rotor, we would like the visual to also show up in the
+    URDF file so that we can see some propellers in rviz. This is why we first
+    have a URDF-specified link and joint, followed by a repetition located
+    inside the <gazebo> tags. -->
+    <link name='rotor_1'>
+      <visual>
+        <geometry>
+            <cylinder length="0.01" radius="0.1"/>
+        </geometry>
+      </visual>
+      <inertial>
+        <mass value="0.005" />
+        <inertia
+          ixx="9.75e-07" ixy="0.0" ixz="0.0"
+          iyy="0.000273104" iyz="0.0"
+          izz="0.000274004"/>
+      </inertial>
+      <pose>-0.13 0.2 0.023 0 0 0</pose>
+      <collision name='rotor_1_collision'>
+        <pose>0 0 0 0 0 0</pose>
+        <geometry>
+          <cylinder>
+            <length>0.005</length>
+            <radius>0.128</radius>
+          </cylinder>
+        </geometry>
+        <surface>
+          <contact> <ode/> </contact>
+          <friction> <ode/> </friction>
+        </surface>
+      </collision>
+    </link>
+    <joint name="rotor_1_joint" type="revolute">
+      <origin xyz="-0.13 0.2 0.023" rpy="0 0 0"/>
+      <parent link="base_link"/>
+      <child link="rotor_1"/>
+      <axis xyz="0 0 1"/>
+      <limit lower="-1e+16" upper="+1e+16" effort="0" velocity="0"/>
+    </joint>
+    <gazebo reference="rotor_1">
+      <gravity>1</gravity>
+      <visual name='rotor_1_visual'>
+          <pose>0 0 0 0 0 0</pose>
+          <geometry>
+              <mesh>
+                  <scale>1 1 1</scale>
+                  <uri>$(find ifo_description)/meshes/iris_prop_cw.dae</uri>
+              </mesh>
+          </geometry>
+          <material>
+              <script>
+                  <name>Gazebo/DarkGrey</name>
+                  <uri>file://media/materials/scripts/gazebo.material</uri>
+              </script>
+          </material>
+      </visual>
+      <velocity_decay/>
+    </gazebo>
+    <gazebo reference="rotor_1_joint">
+      <dynamics>
+          <spring_reference>0</spring_reference>
+          <spring_stiffness>0</spring_stiffness>
+      </dynamics>
+      <use_parent_model_frame>1</use_parent_model_frame>
+    </gazebo>
+    <!-- ===================================================================== -->
+    <!--                               ROTOR 2                                 -->
+    <!-- ===================================================================== -->
+    <!-- For each rotor, we would like the visual to also show up in the
+    URDF file so that we can see some propellers in rviz. This is why we first
+    have a URDF-specified link and joint, followed by a repetition located
+    inside the <gazebo> tags. -->
+    <link name='rotor_2'>
+      <visual>
+        <geometry>
+            <cylinder length="0.01" radius="0.1"/>
+        </geometry>
+      </visual>
+      <inertial>
+        <mass value="0.005" />
+        <inertia
+        ixx="9.75e-07" ixy="0.0" ixz="0.0"
+        iyy="0.000273104" iyz="0.0"
+        izz="0.000274004"/>
+      </inertial>
+      <pose>0.13 0.22 0.023 0 0 0</pose>
+      <collision name='rotor_2_collision'>
+        <pose>0 0 0 0 0 0</pose>
+        <geometry>
+          <cylinder>
+            <length>0.005</length>
+            <radius>0.128</radius>
+          </cylinder>
+        </geometry>
+        <surface>
+        <contact>
+          <ode/>
+        </contact>
+        <friction>
+          <ode/>
+        </friction>
+        </surface>
+      </collision>
+    </link>
+    <joint name="rotor_2_joint" type="revolute">
+      <origin xyz="0.13 0.22 0.023" rpy="0 0 0"/>
+      <parent link="base_link"/>
+      <child link="rotor_2"/>
+      <axis xyz="0 0 1"/>
+      <limit lower="-1e+16" upper="+1e+16" effort="0" velocity="0"/>
+    </joint>
+    <gazebo reference="rotor_2">
+      <gravity>1</gravity>
+      <visual name='rotor_2_visual'>
+          <pose>0 0 0 0 0 0</pose>
+          <geometry>
+              <mesh>
+                  <scale>1 1 1</scale>
+                  <uri>$(find ifo_description)/meshes/iris_prop_cw.dae</uri>
+              </mesh>
+          </geometry>
+          <material>
+              <script>
+                  <name>Gazebo/Blue</name>
+                  <uri>file://media/materials/scripts/gazebo.material</uri>
+              </script>
+          </material>
+      </visual>
+      <velocity_decay/>
+    </gazebo>
+    <gazebo reference="rotor_2_joint">
+      <dynamics>
+          <spring_reference>0</spring_reference>
+          <spring_stiffness>0</spring_stiffness>
+      </dynamics>
+      <use_parent_model_frame>1</use_parent_model_frame>
+    </gazebo>
+    <!-- ===================================================================== -->
+    <!--                               ROTOR 3                                 -->
+    <!-- ===================================================================== -->
+    <!-- For each rotor, we would like the visual to also show up in the
+    URDF file so that we can see some propellers in rviz. This is why we first
+    have a URDF-specified link and joint, followed by a repetition located
+    inside the <gazebo> tags. -->
+    <link name='rotor_3'>
+      <visual>
+        <geometry>
+          <cylinder length="0.01" radius="0.1"/>
+        </geometry>
+      </visual>
+      <inertial>
+          <mass value="0.005" />
+          <inertia
+            ixx="9.75e-07" ixy="0.0" ixz="0.0"
+            iyy="0.000273104" iyz="0.0"
+            izz="0.000274004"/>
+      </inertial>
+      <pose>-0.13 -0.2 0.023 0 0 0</pose>
+        <collision>
           <pose>0 0 0 0 0 0</pose>
           <geometry>
@@ -110,226 +308,5 @@
           </surface>
         </collision>
-        <visual name='rotor_0_visual'>
-          <pose>0 0 0 0 0 0</pose>
-          <geometry>
-            <mesh>
-              <scale>1 1 1</scale>
-              <uri>$(find ifo_description)/meshes/iris_prop_ccw.dae</uri>
-            </mesh>
-          </geometry>
-          <material>
-            <script>
-              <name>Gazebo/Blue</name>
-              <uri>file://media/materials/scripts/gazebo.material</uri>
-            </script>
-          </material>
-        </visual>
-        <gravity>1</gravity>
         <velocity_decay/>
-      </link>
-      <joint name='rotor_0_joint' type='revolute'>
-        <child>rotor_0</child>
-        <parent>base_link</parent>
-        <axis>
-          <xyz>0 0 1</xyz>
-          <limit>
-            <lower>-1e+16</lower>
-            <upper>1e+16</upper>
-          </limit>
-          <dynamics>
-            <spring_reference>0</spring_reference>
-            <spring_stiffness>0</spring_stiffness>
-          </dynamics>
-          <use_parent_model_frame>1</use_parent_model_frame>
-        </axis>
-      </joint>
-    </gazebo>
-    <!-- ===================================================================== -->
-    <!--                               ROTOR 1                                 -->
-    <!-- ===================================================================== -->
-    <!-- For each rotor, we would like the visual to also show up in the
-    URDF file so that we can see some propellers in rviz. This is why we first
-    have a URDF-specified link and joint, followed by a repetition located
-    inside the <gazebo> tags. -->
-    <link name='rotor_1'>
-      <visual>
-        <geometry>
-          <cylinder length="0.01" radius="0.1"/>
-        </geometry>
-      </visual>
-    </link>
-    <joint name="rotor_1_joint" type="revolute">
-      <origin xyz="-0.13 0.2 0.023" rpy="0 0 0"/>
-      <parent link="base_link"/>
-      <child link="rotor_1"/>
-      <axis xyz="0 0 1"/>
-      <limit lower="-1e+16" upper="+1e+16" effort="0" velocity="0"/>
-    </joint>
-    <gazebo>
-      <link name='rotor_1'>
-        <pose>-0.13 0.2 0.023 0 0 0</pose>
-        <inertial>
-          <mass>0.005</mass>
-          <inertia>
-            <ixx>9.75e-07</ixx>
-            <ixy>0</ixy>
-            <ixz>0</ixz>
-            <iyy>0.000273104</iyy>
-            <iyz>0</iyz>
-            <izz>0.000274004</izz>
-          </inertia>
-        </inertial>
-        <collision name='rotor_1_collision'>
-          <pose>0 0 0 0 0 0</pose>
-          <geometry>
-            <cylinder>
-              <length>0.005</length>
-              <radius>0.128</radius>
-            </cylinder>
-          </geometry>
-          <surface>
-            <contact>
-              <ode/>
-            </contact>
-            <friction>
-              <ode/>
-            </friction>
-          </surface>
-        </collision>
-        <visual name='rotor_1_visual'>
-          <pose>0 0 0 0 0 0</pose>
-          <geometry>
-            <mesh>
-              <scale>1 1 1</scale>
-              <uri>$(find ifo_description)/meshes/iris_prop_ccw.dae</uri>
-            </mesh>
-          </geometry>
-          <material>
-            <script>
-              <name>Gazebo/DarkGrey</name>
-              <uri>file://media/materials/scripts/gazebo.material</uri>
-            </script>
-          </material>
-        </visual>
-        <gravity>1</gravity>
-        <velocity_decay/>
-      </link>
-      <joint name='rotor_1_joint' type='revolute'>
-        <child>rotor_1</child>
-        <parent>base_link</parent>
-        <axis>
-          <xyz>0 0 1</xyz>
-          <limit>
-            <lower>-1e+16</lower>
-            <upper>1e+16</upper>
-          </limit>
-          <dynamics>
-            <spring_reference>0</spring_reference>
-            <spring_stiffness>0</spring_stiffness>
-          </dynamics>
-          <use_parent_model_frame>1</use_parent_model_frame>
-        </axis>
-      </joint>
-    </gazebo>
-    <!-- ===================================================================== -->
-    <!--                               ROTOR 2                                 -->
-    <!-- ===================================================================== -->
-    <!-- For each rotor, we would like the visual to also show up in the
-    URDF file so that we can see some propellers in rviz. This is why we first
-    have a URDF-specified link and joint, followed by a repetition located
-    inside the <gazebo> tags. -->
-    <link name='rotor_2'>
-      <visual>
-        <geometry>
-          <cylinder length="0.01" radius="0.1"/>
-        </geometry>
-      </visual>
-    </link>
-    <joint name="rotor_2_joint" type="revolute">
-      <origin xyz="0.13 0.22 0.023" rpy="0 0 0"/>
-      <parent link="base_link"/>
-      <child link="rotor_2"/>
-      <axis xyz="0 0 1"/>
-      <limit lower="-1e+16" upper="+1e+16" effort="0" velocity="0"/>
-    </joint>
-    <gazebo>
-      <link name='rotor_2'>
-        <pose>0.13 0.22 0.023 0 0 0</pose>
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
File: ifo_description/urdf/realsense_d435i.xacro (robot description, xacro)
@@ -113,7 +113,8 @@
       </imu>
       <plugin filename="libgazebo_ros_imu_sensor.so" name="imu_plugin">
-        <robotNamespace></robotNamespace>
+        <robotNamespace/>
         <topicName>${name}/imu</topicName>
         <bodyName>${name}_link</bodyName>
+        <gaussianNoise>0.0</gaussianNoise>
         <updateRateHZ>100.0</updateRateHZ>
         <xyzOffset>0 0 0</xyzOffset>
@@ -283,5 +284,5 @@
   <!-- ________________________ Realsense PLUGIN  _________________________-->
   <gazebo>
-    <plugin name="/${name}" filename="librealsense_gazebo_plugin.so">
+    <plugin name="${name}" filename="librealsense_gazebo_plugin.so">
       <prefix>${name}_</prefix>
       <!-- Color camera settings-->
